Commit message: new plots for 29 grams instead of 27

File: gym-pybullet-drones/gym_pybullet_drones/assets/cf2p.urdf (robot description, URDF)
Before this commit: robot cf2, 6 links, 5 joints
Links:
- link base_link: mass 0.027 -> 0.029

File: gym-pybullet-drones/gym_pybullet_drones/assets/cf2x.urdf (robot description, URDF)
Before this commit: robot cf2, 6 links, 5 joints
Links:
- link base_link: mass 0.027 -> 0.029
